File: pcb/main.brd (EAGLE design)
At the start: 355.6 x 153.3 mm, 222 parts

Commit message: updated schematic for main board
Parts:
- removed C13, C14, C15, C16, C17, C18, C19, C20, C21, C22, C23, C24, C25, C26, C27, C28, C29, C30, C31, C32, C33, C34, C35, C36, C37, C38, C39, C40, C41, C42, C43, C44, C45, C46, C47, C48, C49, C50, C51, C52, C53, C54, C55, C56, C57, C58, C59, C60, C61, C62, C63, C64, C65, C66, C67, C68: (no value), rcl:C1206
- removed C69, C71, C72: (no value), rcl:153CLV-0605
- removed LED1, LED10, LED100, LED101, LED102, LED103, LED104, LED105, LED106, LED107, LED108, LED109, LED11, LED110, LED111, LED112, LED113, LED114, LED115, LED116, LED117, LED118, LED119, LED12, LED120, LED121, LED122, LED123, LED124, LED125, LED126, LED127, LED128, LED129, LED13, LED14, LED15, LED16, LED17, LED18, LED19, LED2, LED20, LED21, LED22, LED23, LED24, LED25, LED26, LED27, LED28, LED29, LED3, LED30, LED31, LED32, LED33, LED34, LED35, LED36, LED37, LED38, LED39, LED4, LED40, LED41, LED42, LED43, LED44, LED45, LED46, LED47, LED48, LED49, LED5, LED50, LED51, LED52, LED53, LED54, LED55, LED56, LED57, LED58, LED59, LED6, LED60, LED61, LED62, LED63, LED64, LED65, LED66, LED67, LED68, LED69, LED7, LED70, LED71, LED72, LED73, LED74, LED75, LED76, LED77, LED78, LED79, LED8, LED80, LED81, LED82, LED83, LED84, LED85, LED86, LED87, LED88, LED89, LED9, LED90, LED91, LED92, LED93, LED94, LED95, LED96, LED97, LED98, LED99: APA102, adafruit:APA102
- removed R49, R50, R51, R52: 10k, rcl:M1206
- removed R53, R56: 120R, rcl:M1206
- removed R55: 390R, rcl:M1206
- removed SL1: (no value), con-amp-quick:06P
- removed SL2: (no value), con-amp-quick:02P
- removed U$12, U$13, U$14, U$15, U$16: 74HCT125D, SparkFun-DigitalIC:SO014
- added C4: (no value), rcl:E3,5-8
- added D1: 1N5400, diode:DO201-15
- added IC2, IC3, IC4: 74HCT04N, 74xx-eu:DIL14
- added U$5: DCDC, main:DCDC
- added U$6: ESP32DEVKITV1, ESP32-DEVKITV1:ESP32-DEVKITV1
- added U$7, U$8: LEDCON, main:LEDCON
- C1, C6, C7: device rcl:153CLV-0605 -> rcl:E3,5-8
- C10, C11, C3, C9: device rcl:C1206 -> rcl:E3,5-8
- C12, C2, C5: device rcl:C1206 -> rcl:C025_050-025X075
- C8: device rcl:153CLV-0405 -> rcl:C025_050-025X075
- IC1: value (none) -> 74HCT04N; device v-reg:317TS -> 74xx-eu:DIL14
- U$1: value ESP07-16PIN -> DCDC; device esp8266modules:ESP07-16PIN -> main:DCDC
- U$10, U$9: value 74HCT125D -> LEDCON; device SparkFun-DigitalIC:SO014 -> main:LEDCON
- U$11: value 74HCT125D -> TX30; device SparkFun-DigitalIC:SO014 -> main:XT30
- U$2: value CMODS6 -> CMODS6TH
- moved C12 419.3 mm to (-226.6, -388.4), flipped to the top, turned to 0 degrees
- moved U$9 371.2 mm to (-222.2, -317.0), flipped to the top, turned to 0 degrees
- moved U$10 370.0 mm to (-222.2, -349.5), flipped to the top, turned to 0 degrees
- moved C8 355.6 mm to (-226.6, -383.5), flipped to the top, turned to 0 degrees
- moved C2 350.9 mm to (-226.6, -373.9), flipped to the top, turned to 0 degrees
- moved C5 350.7 mm to (-226.6, -378.7), flipped to the top, turned to 0 degrees
- moved U$11 290.7 mm to (-223.8, -395.7)
- moved C11 258.9 mm to (-192.8, -223.5), flipped to the top, turned to 0 degrees
- moved C10 249.0 mm to (-192.8, -214.9), flipped to the top, turned to 0 degrees
- moved C9 239.1 mm to (-192.8, -206.2), flipped to the top, turned to 0 degrees
- moved IC1 235.5 mm to (-185.9, -267.0), flipped to the top, turned to 0 degrees
- moved C3 168.6 mm to (-192.8, -163.1)
- moved C6 142.7 mm to (-192.8, -180.3), flipped to the top, turned to 0 degrees
- moved C7 141.2 mm to (-192.8, -189.0), flipped to the top, turned to 0 degrees
- moved U$1 123.8 mm to (-196.1, -105.7), turned to 0 degrees
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Connections:
- removed net +3V3: C3.1, C5.1, C8.+, IC1.2, R49.2, R51.2, R52.2, R53.2, U$1.VCC
- removed net GA1: U$2.P$8, U$9.2
- removed net GA2: U$2.P$9, U$9.5
- removed net GA3: U$2.P$10, U$9.9
- removed net GA4: U$2.P$11, U$9.12
- removed net GA5: U$10.2, U$2.P$12
- removed net GA6: U$10.5, U$2.P$13
- removed net GA7: U$10.9, U$2.P$14
- removed net GA8: U$10.12, U$2.P$15
- removed net GB1: U$11.2, U$2.P$33
- removed net GB2: U$11.5, U$2.P$32
- removed net GB3: U$11.9, U$2.P$31
- removed net GB4: U$11.12, U$2.P$30
- removed net GB5: U$12.2, U$2.P$16
- removed net GB6: U$12.5, U$2.P$17
- removed net GB7: U$12.9, U$2.P$18
- removed net GB8: U$12.12, U$2.P$19
- removed net GC1: U$13.2, U$2.P$29
- removed net GC2: U$13.5, U$2.P$28
- removed net GC3: U$13.9, U$2.P$27
- removed net GC4: U$13.12, U$2.P$26
- removed net GC5: U$14.2, U$2.P$20
- removed net GC6: U$14.5, U$2.P$21
- removed net GC7: U$14.9, U$2.P$22
- removed net GC8: U$14.12, U$2.P$23
- removed net GD1: U$15.2, U$2.P$41
- removed net GD2: U$15.5, U$2.P$40
- removed net GD3: U$15.9, U$2.P$39
- removed net GD4: U$15.12, U$2.P$38
- removed net GD5: U$16.2, U$2.P$37
- removed net GD6: U$16.5, U$2.P$36
- removed net GD7: U$16.9, U$2.P$35
- removed net GD8: U$16.12, U$2.P$34
- removed net GPIO0: R51.1, SL1.1, U$1.GPIO0, U$2.P$5
- removed net GPIO12: U$1.GPIO12, U$2.P$46
- removed net GPIO13: U$1.GPIO13, U$2.P$45
- removed net GPIO14: U$1.GPIO14, U$2.P$47
- removed net GPIO15: R50.2, U$1.GPIO15, U$2.P$7
- removed net GPIO16: U$1.GPIO16, U$2.P$48
- removed net GPIO2: U$1.GPIO2, U$2.P$6
- removed net GPIO4: U$1.GPIO4, U$2.P$3
- removed net GPIO5: U$1.GPIO5, U$2.P$4
- removed net N$100: LED23.DO, LED24.DI
- removed net N$101: LED23.CO, LED24.CI
- removed net N$102: LED20.DO, LED21.DI
- removed net N$103: LED20.CO, LED21.CI
- removed net N$104: LED35.DO, LED36.DI
- removed net N$105: LED24.DO, LED25.DI
- removed net N$106: LED24.CO, LED25.CI
- removed net N$107: LED25.DO, LED26.DI
- removed net N$108: LED25.CO, LED26.CI
- removed net N$109: LED26.DO, LED27.DI
- removed net N$112: LED26.CO, LED27.CI
- removed net N$113: LED27.DO, LED28.DI
- removed net N$114: LED27.CO, LED28.CI
- removed net N$115: LED28.DO, LED29.DI
- removed net N$116: IC1.1, R55.2, R56.1
- removed net N$117: LED28.CO, LED29.CI
- removed net N$118: R53.1, R56.2
- removed net N$119: LED29.DO, LED30.DI
- removed net N$120: LED29.CO, LED30.CI
- removed net N$123: LED1.DI, U$9.3
- removed net N$162: LED30.DO, LED31.DI
- removed net N$163: LED30.CO, LED31.CI
- removed net N$164: LED31.DO, LED32.DI
- removed net N$165: LED31.CO, LED32.CI
- removed net N$166: LED32.DO, LED33.DI
- removed net N$167: LED32.CO, LED33.CI
- removed net N$168: LED1.CI, U$9.6
- removed net N$169: LED6.DI, U$9.8
- removed net N$170: LED6.CI, U$9.11
- removed net N$171: LED12.DI, U$10.3
- removed net N$172: LED12.CI, U$10.6
- removed net N$173: LED20.DI, U$10.8
- removed net N$174: LED20.CI, U$10.11
- removed net N$180: LED35.CO, LED36.CI
- removed net N$181: LED36.DO, LED37.DI
- removed net N$183: LED36.CO, LED37.CI
- removed net N$184: LED37.DO, LED38.DI
- removed net N$185: LED37.CO, LED38.CI
- removed net N$186: LED34.DO, LED35.DI
- removed net N$187: LED34.CO, LED35.CI
- removed net N$188: LED40.DO, LED41.DI
- removed net N$189: LED40.CO, LED41.CI
- removed net N$190: LED41.DO, LED42.DI
- removed net N$191: LED41.CO, LED42.CI
- removed net N$192: LED42.DO, LED43.DI
- removed net N$193: LED42.CO, LED43.CI
- removed net N$194: LED39.DO, LED40.DI
- removed net N$195: LED39.CO, LED40.CI
- removed net N$196: LED43.DO, LED44.DI
- removed net N$197: LED43.CO, LED44.CI
- removed net N$198: LED46.DO, LED47.DI
- removed net N$199: LED46.CO, LED47.CI
- removed net N$200: LED47.DO, LED48.DI
- removed net N$201: LED47.CO, LED48.CI
- removed net N$202: LED48.DO, LED49.DI
- removed net N$203: LED48.CO, LED49.CI
- removed net N$204: LED45.DO, LED46.DI
- removed net N$205: LED45.CO, LED46.CI
- removed net N$206: LED49.DO, LED50.DI
- removed net N$207: LED49.CO, LED50.CI
- removed net N$208: LED50.DO, LED51.DI
- removed net N$209: LED50.CO, LED51.CI
- removed net N$210: LED51.DO, LED52.DI
- removed net N$211: LED51.CO, LED52.CI
- removed net N$212: LED54.DO, LED55.DI
- removed net N$213: LED54.CO, LED55.CI
- removed net N$214: LED55.DO, LED56.DI
- removed net N$215: LED55.CO, LED56.CI
- removed net N$216: LED56.DO, LED57.DI
- removed net N$217: LED56.CO, LED57.CI
- removed net N$218: LED53.DO, LED54.DI
- removed net N$219: LED53.CO, LED54.CI
- removed net N$220: LED57.DO, LED58.DI
- removed net N$221: LED57.CO, LED58.CI
- removed net N$222: LED58.DO, LED59.DI
- removed net N$223: LED58.CO, LED59.CI
- removed net N$224: LED59.DO, LED60.DI
- removed net N$225: LED59.CO, LED60.CI
- removed net N$226: LED60.DO, LED61.DI
- removed net N$227: LED60.CO, LED61.CI
- removed net N$228: LED61.DO, LED62.DI
- removed net N$229: LED61.CO, LED62.CI
- removed net N$230: LED62.DO, LED63.DI
- removed net N$231: LED62.CO, LED63.CI
- removed net N$232: LED63.DO, LED64.DI
- removed net N$233: LED63.CO, LED64.CI
- removed net N$234: LED64.DO, LED65.DI
- removed net N$235: LED64.CO, LED65.CI
- removed net N$236: LED67.DO, LED68.DI
- removed net N$237: LED67.CO, LED68.CI
- removed net N$238: LED34.DI, U$11.3
- removed net N$239: LED34.CI, U$11.6
- removed net N$240: LED39.DI, U$11.8
- removed net N$241: LED39.CI, U$11.11
- removed net N$242: LED45.DI, U$12.3
- removed net N$243: LED45.CI, U$12.6
- removed net N$244: LED53.DI, U$12.8
- removed net N$245: LED53.CI, U$12.11
- removed net N$255: LED68.DO, LED69.DI
- removed net N$256: LED68.CO, LED69.CI
- removed net N$257: LED69.DO, LED70.DI
- removed net N$258: LED69.CO, LED70.CI
- removed net N$259: LED66.DO, LED67.DI
- removed net N$260: LED66.CO, LED67.CI
- removed net N$261: LED72.DO, LED73.DI
- removed net N$262: LED72.CO, LED73.CI
- removed net N$263: LED73.DO, LED74.DI
- removed net N$264: LED73.CO, LED74.CI
- removed net N$265: LED74.DO, LED75.DI
- removed net N$266: LED74.CO, LED75.CI
- removed net N$267: LED71.DO, LED72.DI
- removed net N$268: LED71.CO, LED72.CI
- removed net N$269: LED75.DO, LED76.DI
- removed net N$270: LED75.CO, LED76.CI
- removed net N$271: LED78.DO, LED79.DI
- removed net N$272: LED78.CO, LED79.CI
- removed net N$273: LED79.DO, LED80.DI
- removed net N$274: LED79.CO, LED80.CI
- removed net N$275: LED80.DO, LED81.DI
- removed net N$276: LED80.CO, LED81.CI
- removed net N$277: LED77.DO, LED78.DI
- removed net N$278: LED77.CO, LED78.CI
- removed net N$279: LED81.DO, LED82.DI
- removed net N$280: LED81.CO, LED82.CI
- removed net N$281: LED82.DO, LED83.DI
- removed net N$282: LED82.CO, LED83.CI
- removed net N$283: LED83.DO, LED84.DI
- removed net N$284: LED83.CO, LED84.CI
- removed net N$285: LED86.DO, LED87.DI
- removed net N$286: LED86.CO, LED87.CI
- removed net N$287: LED87.DO, LED88.DI
- removed net N$288: LED87.CO, LED88.CI
- removed net N$289: LED88.DO, LED89.DI
- removed net N$290: LED88.CO, LED89.CI
- removed net N$291: LED85.DO, LED86.DI
- removed net N$292: LED85.CO, LED86.CI
- removed net N$293: LED89.DO, LED90.DI
- removed net N$294: LED89.CO, LED90.CI
- removed net N$295: LED90.DO, LED91.DI
- removed net N$296: LED90.CO, LED91.CI
- removed net N$297: LED91.DO, LED92.DI
- removed net N$298: LED91.CO, LED92.CI
- removed net N$299: LED92.DO, LED93.DI
- removed net N$300: LED92.CO, LED93.CI
- removed net N$301: LED93.DO, LED94.DI
- removed net N$302: LED93.CO, LED94.CI
- removed net N$303: LED94.DO, LED95.DI
- removed net N$304: LED94.CO, LED95.CI
- removed net N$305: LED95.DO, LED96.DI
- removed net N$306: LED95.CO, LED96.CI
- removed net N$307: LED96.DO, LED97.DI
- removed net N$308: LED96.CO, LED97.CI
- removed net N$309: LED66.DI, U$13.3
- removed net N$310: LED66.CI, U$13.6
- removed net N$311: LED71.DI, U$13.8
- removed net N$312: LED71.CI, U$13.11
- removed net N$313: LED77.DI, U$14.3
- removed net N$314: LED77.CI, U$14.6
- removed net N$315: LED85.DI, U$14.8
- removed net N$316: LED85.CI, U$14.11
- removed net N$326: LED100.DI, LED99.DO
- removed net N$327: LED100.CI, LED99.CO
- removed net N$328: LED100.DO, LED101.DI
- removed net N$329: LED100.CO, LED101.CI
- removed net N$330: LED101.DO, LED102.DI
- removed net N$331: LED101.CO, LED102.CI
- removed net N$332: LED98.DO, LED99.DI
- removed net N$333: LED98.CO, LED99.CI
- removed net N$334: LED104.DO, LED105.DI
- removed net N$335: LED104.CO, LED105.CI
- removed net N$336: LED105.DO, LED106.DI
- removed net N$337: LED105.CO, LED106.CI
- removed net N$338: LED106.DO, LED107.DI
- removed net N$339: LED106.CO, LED107.CI
- removed net N$340: LED103.DO, LED104.DI
- removed net N$341: LED103.CO, LED104.CI
- removed net N$342: LED107.DO, LED108.DI
- removed net N$343: LED107.CO, LED108.CI
- removed net N$344: LED110.DO, LED111.DI
- removed net N$345: LED110.CO, LED111.CI
- removed net N$346: LED111.DO, LED112.DI
- removed net N$347: LED111.CO, LED112.CI
- removed net N$348: LED112.DO, LED113.DI
- removed net N$349: LED112.CO, LED113.CI
- removed net N$350: LED109.DO, LED110.DI
- removed net N$351: LED109.CO, LED110.CI
- removed net N$352: LED113.DO, LED114.DI
- removed net N$353: LED113.CO, LED114.CI
- removed net N$354: LED114.DO, LED115.DI
- removed net N$355: LED114.CO, LED115.CI
- removed net N$356: LED115.DO, LED116.DI
- removed net N$357: LED115.CO, LED116.CI
- removed net N$358: LED118.DO, LED119.DI
- removed net N$359: LED118.CO, LED119.CI
- removed net N$360: LED119.DO, LED120.DI
- removed net N$361: LED119.CO, LED120.CI
- removed net N$362: LED120.DO, LED121.DI
- removed net N$363: LED120.CO, LED121.CI
- removed net N$364: LED117.DO, LED118.DI
- removed net N$365: LED117.CO, LED118.CI
- removed net N$366: LED121.DO, LED122.DI
- removed net N$367: LED121.CO, LED122.CI
- removed net N$368: LED122.DO, LED123.DI
- removed net N$369: LED122.CO, LED123.CI
- removed net N$370: LED123.DO, LED124.DI
- removed net N$371: LED123.CO, LED124.CI
- removed net N$372: LED124.DO, LED125.DI
- removed net N$373: LED124.CO, LED125.CI
- removed net N$374: LED125.DO, LED126.DI
- removed net N$375: LED125.CO, LED126.CI
- removed net N$376: LED126.DO, LED127.DI
- removed net N$377: LED126.CO, LED127.CI
- removed net N$378: LED127.DO, LED128.DI
- removed net N$379: LED127.CO, LED128.CI
- removed net N$380: LED128.DO, LED129.DI
- removed net N$381: LED128.CO, LED129.CI
- removed net N$382: LED98.DI, U$15.3
- removed net N$383: LED98.CI, U$15.6
- removed net N$384: LED103.DI, U$15.8
- removed net N$385: LED103.CI, U$15.11
- removed net N$386: LED109.DI, U$16.3
- removed net N$387: LED109.CI, U$16.6
- removed net N$388: LED117.DI, U$16.8
- removed net N$389: LED117.CI, U$16.11
- removed net N$46: LED2.DO, LED3.DI
- removed net N$51: LED2.CO, LED3.CI
- removed net N$56: LED3.DO, LED4.DI
- removed net N$57: LED3.CO, LED4.CI
- removed net N$58: LED4.DO, LED5.DI
- removed net N$59: LED4.CO, LED5.CI
- removed net N$60: LED1.DO, LED2.DI
- removed net N$61: LED1.CO, LED2.CI
- removed net N$66: LED7.DO, LED8.DI
- removed net N$67: LED7.CO, LED8.CI
- removed net N$68: LED8.DO, LED9.DI
- removed net N$69: LED8.CO, LED9.CI
- removed net N$70: LED10.DI, LED9.DO
- removed net N$71: LED10.CI, LED9.CO
- removed net N$72: LED6.DO, LED7.DI
- removed net N$73: LED6.CO, LED7.CI
- removed net N$75: LED10.DO, LED11.DI
- removed net N$76: LED10.CO, LED11.CI
- removed net N$77: LED21.DO, LED22.DI
- removed net N$78: LED13.DO, LED14.DI
- removed net N$80: LED13.CO, LED14.CI
- removed net N$82: LED14.DO, LED15.DI
- removed net N$83: R52.1, SL1.5, U$1.REST
- removed net N$84: R49.1, U$1.CH_PD
- removed net N$85: LED14.CO, LED15.CI
- removed net N$86: LED15.DO, LED16.DI
- removed net N$87: LED15.CO, LED16.CI
- removed net N$88: LED12.DO, LED13.DI
- removed net N$89: LED12.CO, LED13.CI
- removed net N$91: LED16.DO, LED17.DI
- removed net N$92: LED16.CO, LED17.CI
- removed net N$93: LED21.CO, LED22.CI
- removed net N$94: LED17.DO, LED18.DI
- removed net N$95: LED17.CO, LED18.CI
- removed net N$96: LED22.DO, LED23.DI
- removed net N$97: LED18.DO, LED19.DI
- removed net N$98: LED18.CO, LED19.CI
- removed net N$99: LED22.CO, LED23.CI
- removed net RX: SL1.3, U$1.RX, U$2.P$2
- removed net TX: SL1.2, U$1.TX, U$2.P$1
- new net +5V/3: C10.+, C8.1, IC3.14, U$4.VOUT1, U$4.VOUT2
- new net +5V/4: C11.+, C12.1, IC4.14, U$5.VOUT1, U$5.VOUT2
- new net C1: IC1.11, IC1.13, U$2.14
- new net C2: IC2.11, IC2.13, U$2.19
- new net C3: IC3.11, IC3.13, U$2.35
- new net C4: IC4.11, IC4.13, U$2.30
- new net D11: IC1.1, U$2.15
- new net D12: IC1.3, U$2.16
- new net D13: IC1.5, U$2.17
- new net D14: IC1.9, U$2.18
- new net D21: IC2.1, U$2.20
- new net D22: IC2.3, U$2.21
- new net D23: IC2.5, U$2.22
- new net D24: IC2.9, U$2.23
- new net D31: IC3.1, U$2.34
- new net D32: IC3.3, U$2.33
- new net D33: IC3.5, U$2.32
- new net D34: IC3.9, U$2.31
- new net D41: IC4.1, U$2.29
- new net D42: IC4.3, U$2.28
- new net D43: IC4.5, U$2.27
- new net D44: IC4.9, U$2.26
- new net IO13: U$2.48, U$6.28
- new net IO14: U$2.47, U$6.26
- new net IO15: U$2.1, U$6.3
- new net IO16: U$2.3, U$6.6
- new net IO17: U$2.4, U$6.7
- new net IO18: U$2.6, U$6.9
- new net IO19: U$2.7, U$6.10
- new net IO21: U$2.8, U$6.11
- new net IO22: U$2.9, U$6.14
- new net IO23: U$2.10, U$6.15
- new net IO25: U$2.44, U$6.23
- new net IO26: U$2.45, U$6.24
- new net IO27: U$2.46, U$6.24
- new net IO32: U$2.42, U$6.21
- new net IO33: U$2.43, U$6.22
- new net IO4: U$2.2, U$6.5
- new net IO5: U$2.5, U$6.8
- new net N$10: IC2.4, U$8.D2
- new net N$11: IC2.2, U$8.D1
- new net N$12: IC2.10, U$8.C3, U$8.C4
- new net N$13: IC2.12, U$8.C1, U$8.C2
- new net N$14: IC3.8, U$9.D4
- new net N$15: IC3.6, U$9.D3
- new net N$16: IC3.4, U$9.D2
- new net N$17: IC3.2, U$9.D1
- new net N$18: IC3.10, U$9.C3, U$9.C4
- new net N$19: IC3.12, U$9.C1, U$9.C2
- new net N$2: IC1.8, U$7.D4
- new net N$20: IC4.8, U$10.D4
- new net N$21: IC4.6, U$10.D3
- new net N$22: IC4.4, U$10.D2
- new net N$23: IC4.2, U$10.D1
- new net N$24: IC4.10, U$10.C3, U$10.C4
- new net N$25: IC4.12, U$10.C1, U$10.C2
- new net N$26: D1.A, U$11.P
- new net N$3: IC1.6, U$7.D3
- new net N$4: IC1.4, U$7.D2
- new net N$5: IC1.2, U$7.D1
- new net N$6: IC1.10, U$7.C3, U$7.C4
- new net N$7: IC1.12, U$7.C1, U$7.C2
- new net N$8: IC2.8, U$8.D4
- new net N$9: IC2.6, U$8.D3
- net +12V: now also C3.+, D1.C, SL3.1, U$1.VIN1, U$1.VIN2, U$2.24, U$5.VIN1, U$5.VIN2, U$6.30; no longer C2.1, C69.+, C71.+, C72.+, IC1.3, SL2.2, U$2.P$24
- net +5V/1: now also C2.1, C4.+, IC1.14, U$1.VOUT1, U$1.VOUT2; no longer C10.1, C11.1, C12.1, C13.1, C14.1, C15.1, C16.1, C17.1, C18.1, C19.1, C20.1, C21.1, C22.1, C23.1, C24.1, C25.1, C26.1, C27.1, C28.1, C29.1, C30.1, C31.1, C32.1, C33.1, C34.1, C35.1, C36.1, C37.1, C38.1, C9.1, LED1.VCC, LED10.VCC, LED11.VCC, LED12.VCC, LED13.VCC, LED14.VCC, LED15.VCC, LED16.VCC, LED17.VCC, LED18.VCC, LED19.VCC, LED2.VCC, LED20.VCC, LED21.VCC, LED22.VCC, LED23.VCC, LED24.VCC, LED25.VCC, LED26.VCC, LED27.VCC, LED28.VCC, LED29.VCC, LED3.VCC, LED30.VCC, LED31.VCC, LED32.VCC, LED33.VCC, LED34.VCC, LED35.VCC, LED36.VCC, LED37.VCC, LED38.VCC, LED39.VCC, LED4.VCC, LED40.VCC, LED41.VCC, LED42.VCC, LED43.VCC, LED44.VCC, LED45.VCC, LED46.VCC, LED47.VCC, LED48.VCC, LED49.VCC, LED5.VCC, LED50.VCC, LED51.VCC, LED52.VCC, LED53.VCC, LED54.VCC, LED55.VCC, LED56.VCC, LED57.VCC, LED58.VCC, LED59.VCC, LED6.VCC, LED60.VCC, LED61.VCC, LED62.VCC, LED63.VCC, LED64.VCC, LED65.VCC, LED7.VCC, LED8.VCC, LED9.VCC, SL3.1, U$10.14, U$11.14, U$12.14, U$3.VOUT1, U$3.VOUT2, U$9.14
- net +5V/2: now also C5.1, C9.+, IC2.14, U$3.VOUT1, U$3.VOUT2; no longer C39.1, C40.1, C41.1, C42.1, C43.1, C44.1, C45.1, C46.1, C47.1, C48.1, C49.1, C50.1, C51.1, C52.1, C53.1, C54.1, C55.1, C56.1, C57.1, C58.1, C59.1, C60.1, C61.1, C62.1, C63.1, C64.1, C65.1, C66.1, C67.1, C68.1, LED100.VCC, LED101.VCC, LED102.VCC, LED103.VCC, LED104.VCC, LED105.VCC, LED106.VCC, LED107.VCC, LED108.VCC, LED109.VCC, LED110.VCC, LED111.VCC, LED112.VCC, LED113.VCC, LED114.VCC, LED115.VCC, LED116.VCC, LED117.VCC, LED118.VCC, LED119.VCC, LED120.VCC, LED121.VCC, LED122.VCC, LED123.VCC, LED124.VCC, LED125.VCC, LED126.VCC, LED127.VCC, LED128.VCC, LED129.VCC, LED66.VCC, LED67.VCC, LED68.VCC, LED69.VCC, LED70.VCC, LED71.VCC, LED72.VCC, LED73.VCC, LED74.VCC, LED75.VCC, LED76.VCC, LED77.VCC, LED78.VCC, LED79.VCC, LED80.VCC, LED81.VCC, LED82.VCC, LED83.VCC, LED84.VCC, LED85.VCC, LED86.VCC, LED87.VCC, LED88.VCC, LED89.VCC, LED90.VCC, LED91.VCC, LED92.VCC, LED93.VCC, LED94.VCC, LED95.VCC, LED96.VCC, LED97.VCC, LED98.VCC, LED99.VCC, U$13.14, U$14.14, U$15.14, U$16.14, U$4.VOUT1, U$4.VOUT2
- net GND: now also C10.-, C11.-, C3.-, C4.-, C8.2, C9.-, IC1.7, IC2.7, IC3.7, IC4.7, SL3.2, U$1.GND1, U$1.GND2, U$1.GND3, U$1.GND4, U$11.N, U$2.25, U$5.GND1, U$5.GND2, U$5.GND3, U$5.GND4, U$6.2, U$6.28; no longer C10.2, C11.2, C13.2, C14.2, C15.2, C16.2, C17.2, C18.2, C19.2, C20.2, C21.2, C22.2, C23.2, C24.2, C25.2, C26.2, C27.2, C28.2, C29.2, C3.2, C30.2, C31.2, C32.2, C33.2, C34.2, C35.2, C36.2, C37.2, C38.2, C39.2, C40.2, C41.2, C42.2, C43.2, C44.2, C45.2, C46.2, C47.2, C48.2, C49.2, C50.2, C51.2, C52.2, C53.2, C54.2, C55.2, C56.2, C57.2, C58.2, C59.2, C60.2, C61.2, C62.2, C63.2, C64.2, C65.2, C66.2, C67.2, C68.2, C69.-, C71.-, C72.-, C8.-, C9.2, LED1.GND, LED10.GND, LED100.GND, LED101.GND, LED102.GND, LED103.GND, LED104.GND, LED105.GND, LED106.GND, LED107.GND, LED108.GND, LED109.GND, LED11.GND, LED110.GND, LED111.GND, LED112.GND, LED113.GND, LED114.GND, LED115.GND, LED116.GND, LED117.GND, LED118.GND, LED119.GND, LED12.GND, LED120.GND, LED121.GND, LED122.GND, LED123.GND, LED124.GND, LED125.GND, LED126.GND, LED127.GND, LED128.GND, LED129.GND, LED13.GND, LED14.GND, LED15.GND, LED16.GND, LED17.GND, LED18.GND, LED19.GND, LED2.GND, LED20.GND, LED21.GND, LED22.GND, LED23.GND, LED24.GND, LED25.GND, LED26.GND, LED27.GND, LED28.GND, LED29.GND, LED3.GND, LED30.GND, LED31.GND, LED32.GND, LED33.GND, LED34.GND, LED35.GND, LED36.GND, LED37.GND, LED38.GND, LED39.GND, LED4.GND, LED40.GND, LED41.GND, LED42.GND, LED43.GND, LED44.GND, LED45.GND, LED46.GND, LED47.GND, LED48.GND, LED49.GND, LED5.GND, LED50.GND, LED51.GND, LED52.GND, LED53.GND, LED54.GND, LED55.GND, LED56.GND, LED57.GND, LED58.GND, LED59.GND, LED6.GND, LED60.GND, LED61.GND, LED62.GND, LED63.GND, LED64.GND, LED65.GND, LED66.GND, LED67.GND, LED68.GND, LED69.GND, LED7.GND, LED70.GND, LED71.GND, LED72.GND, LED73.GND, LED74.GND, LED75.GND, LED76.GND, LED77.GND, LED78.GND, LED79.GND, LED8.GND, LED80.GND, LED81.GND, LED82.GND, LED83.GND, LED84.GND, LED85.GND, LED86.GND, LED87.GND, LED88.GND, LED89.GND, LED9.GND, LED90.GND, LED91.GND, LED92.GND, LED93.GND, LED94.GND, LED95.GND, LED96.GND, LED97.GND, LED98.GND, LED99.GND, R50.1, R55.1, SL1.6, SL2.1, SL3.3, U$1.GND, U$10.1, U$10.10, U$10.13, U$10.4, U$10.7, U$11.1, U$11.10, U$11.13, U$11.4, U$11.7, U$12.1, U$12.10, U$12.13, U$12.4, U$12.7, U$13.1, U$13.10, U$13.13, U$13.4, U$13.7, U$14.1, U$14.10, U$14.13, U$14.4, U$14.7, U$15.1, U$15.10, U$15.13, U$15.4, U$15.7, U$16.1, U$16.10, U$16.13, U$16.4, U$16.7, U$2.P$25, U$9.1, U$9.10, U$9.13, U$9.4, U$9.7
- net N$1: now also SL3.3, U$2.36; no longer SL3.2, U$2.P$44
Routing:
- net N$1: track 247.0 -> 0.00 mm, vias 2 -> 0
- net GND: track 328.6 -> 134.1 mm, vias 75 -> 47
- net GA4: track 184.1 -> 0.00 mm
- net GA3: track 172.8 -> 0.00 mm
- net GA2: track 170.1 -> 0.00 mm
- net GA1: track 156.1 -> 0.00 mm
- net GA8: track 140.2 -> 0.00 mm
- net GA7: track 138.8 -> 0.00 mm
- net GA6: track 134.7 -> 0.00 mm
- net GA5: track 113.2 -> 0.00 mm
- net +5V/1: track 115.7 -> 9.40 mm, vias 29 -> 6
- net +12V: track 167.6 -> 76.7 mm
- net GB4: track 71.5 -> 0.00 mm
- net GB2: track 70.5 -> 0.00 mm
- net C4: track 0.00 -> 70.2 mm
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- added copper zone on layer 16, net C1
- added copper zone on layer 16, net C2
- added copper zone on layer 16, net C3
- added copper zone on layer 16, net C4
- added copper zone on layer 16, net D12
- added copper zone on layer 16, net D13
- added copper zone on layer 16, net D14
- added copper zone on layer 16, net D21
- added copper zone on layer 16, net D22
- added copper zone on layer 16, net D23
- added copper zone on layer 16, net D24
- added copper zone on layer 16, net D31
- added copper zone on layer 16, net D32
- added copper zone on layer 16, net D33
- added copper zone on layer 16, net D34
- added copper zone on layer 16, net D41
- added copper zone on layer 16, net D42
- added copper zone on layer 16, net D43
- added copper zone on layer 16, net D44
- removed copper zone on layer 16, net GA7
- removed copper zone on layer 16, net GA8
- removed copper zone on layer 16, net GB1
- removed copper zone on layer 16, net GB2
- removed copper zone on layer 16, net GB3
- removed copper zone on layer 16, net GB4
- removed copper zone on layer 16, net GB5
- removed copper zone on layer 16, net GB6
- removed copper zone on layer 16, net GB7
- removed copper zone on layer 16, net GB8
- removed copper zone on layer 16, net GC1
- removed copper zone on layer 16, net GC2
- removed copper zone on layer 16, net GC3
- removed copper zone on layer 16, net GC4
- removed copper zone on layer 16, net GC5
- removed copper zone on layer 16, net GC6
- removed copper zone on layer 16, net GC7
- removed copper zone on layer 16, net GC8
- removed copper zone on layer 16, net GD7
- removed copper zone on layer 16, net GD8

Commit message: updated schematic for motor driver
Parts:
- added CN1: (no value), microbuilder:DCJACK_2MM_PTH
- added LOGO1: OSHW_LOGO_FILLX0350-NT, ohw-logo:OSHW_FILLX350_NOTEXT
- renumbered SL3 to HALL, U$1 to DCDC1, U$10 to LEDS4, U$11 to POWER, U$2 to CMODS6, U$3 to DCDC2, U$4 to DCDC3, U$5 to DCDC4, U$6 to ESP32, U$7 to LEDS1, U$8 to LEDS2, U$9 to LEDS3
Connections:
- net GND: now also CN1.GND, CN1.GNDBREAK
- net N$26: now also CN1.PWR

Commit message: first version of motor driver pcb layout
Parts:
- removed CN1: (no value), microbuilder:DCJACK_2MM_PTH
- added POWER_TEST: (no value), microbuilder:DCJACK_2MM_PTH
- added U$1: LOGO50MM, im-pro-logo:LOGO_50MM
- CMODS6: device main:DIL48 -> diypov:DIL48
- DCDC1, DCDC2, DCDC3, DCDC4: value DCDC -> DCDC_5V; device main:DCDC -> diypov:DCDC
- HALL: value (none) -> HALL; device con-amp-quick:03P -> diypov:HALL
- LEDS1, LEDS2, LEDS3, LEDS4: device main:LEDCON -> diypov:LEDCON
- POWER: device main:XT30 -> diypov:XT30
- moved C5 531.5 mm to (93.0, 46.0), flipped to the bottom
- moved C2 511.8 mm to (69.3, 43.7), flipped to the bottom
- moved D1 472.7 mm to (26.4, 0.25), flipped to the bottom, turned to 180 degrees
- moved C12 469.5 mm to (63.0, -18.8), flipped to the bottom
- moved C8 469.5 mm to (63.0, -14.0), flipped to the bottom
- moved LOGO1 469.5 mm to (60.5, -46.0)
- moved IC3 454.2 mm to (3.05, 64.5), flipped to the bottom
- moved POWER 443.1 mm to (11.7, -20.3), flipped to the bottom, turned to 270 degrees
- moved IC2 433.2 mm to (75.2, 19.1), flipped to the bottom, turned to 180 degrees
- moved LEDS3 418.7 mm to (0.00, 37.8)
- moved LEDS2 385.8 mm to (38.4, 0.00), turned to 270 degrees
- moved LEDS4 382.6 mm to (0.00, -38.1), turned to 180 degrees
- moved IC4 369.3 mm to (-1.27, -65.8), flipped to the bottom, turned to 180 degrees
- moved LEDS1 321.9 mm to (-37.6, 0.00), turned to 90 degrees
- moved C11 321.3 mm to (-16.3, 45.0), flipped to the bottom
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Connections:
- new net IO1: CMODS6.11, ESP32.13
- new net IO12: CMODS6.47, ESP32.27
- new net IO2: CMODS6.2, ESP32.4
- new net IO3: CMODS6.10, ESP32.12
- new net IO34: CMODS6.39, ESP32.19
- new net IO35: CMODS6.40, ESP32.20
- new net IO36: CMODS6.37, ESP32.17
- new net IO39: CMODS6.38, ESP32.18
- net +12V: now also HALL.VCC; no longer HALL.1
- net GND: now also HALL.GND, POWER_TEST.GND, POWER_TEST.GNDBREAK; no longer CN1.GND, CN1.GNDBREAK, HALL.2
- net IO14: now also CMODS6.46; no longer CMODS6.47
- net IO16: now also CMODS6.4; no longer CMODS6.3
- net IO17: now also CMODS6.5; no longer CMODS6.4
- net IO18: now also CMODS6.7; no longer CMODS6.6
- net IO19: now also CMODS6.8; no longer CMODS6.7
- net IO21: now also CMODS6.9; no longer CMODS6.8
- net IO22: now also CMODS6.12; no longer CMODS6.9
- net IO23: now also CMODS6.13; no longer CMODS6.10
- net IO25: now also CMODS6.43; no longer CMODS6.44
- net IO26: now also CMODS6.44; no longer CMODS6.45
- net IO27: now also CMODS6.45; no longer CMODS6.46
- net IO32: now also CMODS6.41; no longer CMODS6.42
- net IO33: now also CMODS6.42; no longer CMODS6.43
- net IO4: now also CMODS6.3; no longer CMODS6.2
- net IO5: now also CMODS6.6; no longer CMODS6.5
- net N$1: now also HALL.OUT; no longer HALL.3
- net N$26: now also POWER_TEST.PWR; no longer CN1.PWR
Routing:
- net GND: track 134.1 -> 0.00 mm, vias 47 -> 0
- net +5V/2: track 86.9 -> 0.00 mm, vias 2 -> 0
- net +12V: track 76.7 -> 0.00 mm, vias 5 -> 0
- net C4: track 70.2 -> 0.00 mm
- net D33: track 70.2 -> 0.00 mm
- net D32: track 69.7 -> 0.00 mm
- net D34: track 69.2 -> 0.00 mm
- net D11: track 64.9 -> 0.00 mm
- net C1: track 59.7 -> 0.00 mm
- net D12: track 55.6 -> 0.00 mm
- net D13: track 53.5 -> 0.00 mm
- net C2: track 53.0 -> 0.00 mm
- net D14: track 52.2 -> 0.00 mm
- net D41: track 35.7 -> 0.00 mm
- net D42: track 33.4 -> 0.00 mm
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- removed copper zone on layer 1, net +5V/1
- removed copper zone on layer 16, net +5V/1
- removed copper zone on layer 1, net +5V/2
- removed copper zone on layer 16, net +5V/2
- removed copper zone on layer 16, net C1
- removed copper zone on layer 16, net C2
- removed copper zone on layer 16, net C3
- removed copper zone on layer 16, net C4
- removed copper zone on layer 16, net D12
- removed copper zone on layer 16, net D13
- removed copper zone on layer 16, net D14
- removed copper zone on layer 16, net D21
- removed copper zone on layer 16, net D22
- removed copper zone on layer 16, net D23
- removed copper zone on layer 16, net D24
- removed copper zone on layer 16, net D31
- removed copper zone on layer 16, net D32
- removed copper zone on layer 16, net D33
- removed copper zone on layer 16, net D34
- removed copper zone on layer 16, net D41
- removed copper zone on layer 16, net D42
- removed copper zone on layer 16, net D43
- removed copper zone on layer 16, net D44
- removed copper zone on layer 16, net GA1
- removed copper zone on layer 16, net GA2
- removed copper zone on layer 16, net GA3
- removed copper zone on layer 16, net GA4
- removed copper zone on layer 16, net GA5
- removed copper zone on layer 16, net GA6
- removed copper zone on layer 16, net GD1
- removed copper zone on layer 16, net GD2
- removed copper zone on layer 16, net GD3
- removed copper zone on layer 16, net GD4
- removed copper zone on layer 16, net GD5
- removed copper zone on layer 16, net GD6
- removed copper zone on layer 1, net GND
- removed copper zone on layer 16, net GND
- removed copper zone on layer 1, net N$1
- removed copper zone on layer 16, net N$109
- removed copper zone on layer 16, net N$112
- removed copper zone on layer 16, net N$224
- removed copper zone on layer 16, net N$225
- removed copper zone on layer 16, net N$297
- removed copper zone on layer 16, net N$298
- removed copper zone on layer 16, net N$370
- removed copper zone on layer 16, net N$371
Other:
- board size 355.6 x 153.3 mm -> 100 x 100 mm
- board text removed: "Project POV im-pro.at"

Commit message: started layout of main pcb
Parts:
- moved DCDC1 109.1 mm to (-31.5, 26.2)
- moved HALL 102.9 mm to (0.00, -46.5), turned to 0 degrees
- moved C12 98.5 mm to (-35.3, -13.0)
- moved C5 89.6 mm to (24.1, -11.4)
- moved C2 84.8 mm to (-15.2, 37.8)
- moved DCDC2 83.8 mm to (31.5, -26.2), turned to 270 degrees
- moved IC1 82.5 mm to (0.00, 39.6), turned to 180 degrees
- moved DCDC4 78.5 mm to (-31.5, -47.2), turned to 90 degrees
- moved DCDC3 77.7 mm to (31.5, 47.2)
- moved C9 74.7 mm to (33.0, -15.2)
- moved IC4 74.1 mm to (-39.1, -2.03), turned to 90 degrees
- moved IC3 73.8 mm to (38.9, 0.00), turned to 270 degrees
- moved POWER_TEST 73.6 mm to (-13.7, 11.4)
- moved C3 70.6 mm to (-27.4, -12.2)
- moved C10 68.4 mm to (36.1, 17.5), turned to 180 degrees
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Connections:
- net +5V/1: now also LEDS1.VCC
- net +5V/2: now also LEDS2.VCC
- net +5V/3: now also LEDS3.VCC
- net +5V/4: now also LEDS4.VCC
- net GND: now also C12.3, C2.3, C5.3, C8.3, LEDS1.GND, LEDS2.GND, LEDS3.GND, LEDS4.GND
Routing:
- net +12V: track 0.00 -> 532.8 mm
- net +5V/2: track 0.00 -> 112.7 mm
- net +5V/1: track 0.00 -> 75.8 mm
- net +5V/3: track 0.00 -> 52.0 mm
- net +5V/4: track 0.00 -> 51.6 mm
- net N$26: track 0.00 -> 26.9 mm
- added copper zone on layer 1, net GND

Commit message: first version layout main pcb
Parts:
- removed ESP32: ESP32DEVKITV1, ESP32-DEVKITV1:ESP32-DEVKITV1
- added U$2: ESP32DEVKITV1, ESP32-DEVKITV1:ESP32-DEVKITV1
- moved IC4 0.25 mm to (-38.9, -2.03)
Connections:
- removed net IO13: CMODS6.48, ESP32.28
- net +12V: now also U$2.30; no longer ESP32.30
- net C1: now also CMODS6.35; no longer CMODS6.14
- net C2: now also CMODS6.5, IC2.1, IC2.3; no longer CMODS6.19, IC2.11, IC2.13
- net C3: now also CMODS6.48, IC3.1; no longer CMODS6.35, IC3.11
- net C4: now also CMODS6.29; no longer CMODS6.30
- net D11: now also CMODS6.39, IC1.5; no longer CMODS6.15, IC1.1
- net D12: now also CMODS6.37; no longer CMODS6.16
- net D13: now also CMODS6.34, IC1.1; no longer CMODS6.17, IC1.5
- net D14: now also CMODS6.38; no longer CMODS6.18
- net D21: now also CMODS6.4, IC2.5; no longer CMODS6.20, IC2.1
- net D22: now also CMODS6.3, IC2.13; no longer CMODS6.21, IC2.3
- net D23: now also CMODS6.2, IC2.11; no longer CMODS6.22, IC2.5
- net D24: now also CMODS6.1; no longer CMODS6.23
- net D31: now also CMODS6.47, IC3.3; no longer CMODS6.34, IC3.1
- net D32: now also CMODS6.45, IC3.5; no longer CMODS6.33, IC3.3
- net D33: now also CMODS6.46, IC3.11; no longer CMODS6.32, IC3.5
- net D34: now also CMODS6.44; no longer CMODS6.31
- net D41: now also CMODS6.28; no longer CMODS6.29
- net D42: now also CMODS6.27; no longer CMODS6.28
- net D43: now also CMODS6.26; no longer CMODS6.27
- net D44: now also CMODS6.30; no longer CMODS6.26
- net GND: now also U$2.2, U$2.29; no longer ESP32.2, ESP32.28
- net IO1: now also CMODS6.20, U$2.13; no longer CMODS6.11, ESP32.13
- net IO12: now also CMODS6.7, U$2.27; no longer CMODS6.47, ESP32.27
- net IO14: now also CMODS6.8, U$2.26; no longer CMODS6.46, ESP32.26
- net IO15: now also CMODS6.6, U$2.3; no longer CMODS6.1, ESP32.3
- net IO16: now also CMODS6.41, U$2.6; no longer CMODS6.4, ESP32.6
- net IO17: now also CMODS6.40, U$2.7; no longer CMODS6.5, ESP32.7
- net IO18: now also CMODS6.16, U$2.9; no longer CMODS6.7, ESP32.9
- net IO19: now also CMODS6.33, U$2.10; no longer CMODS6.8, ESP32.10
- net IO2: now also CMODS6.43, U$2.4; no longer CMODS6.2, ESP32.4
- net IO21: now also CMODS6.32, U$2.11; no longer CMODS6.9, ESP32.11
- net IO22: now also CMODS6.22, U$2.14; no longer CMODS6.12, ESP32.14
- net IO23: now also CMODS6.23, U$2.15; no longer CMODS6.13, ESP32.15
- net IO25: now also CMODS6.12, U$2.23; no longer CMODS6.43, ESP32.23
- net IO26: now also CMODS6.10, U$2.24; no longer CMODS6.44, ESP32.24
- net IO27: now also CMODS6.9, U$2.25; no longer CMODS6.45, ESP32.24
- net IO3: now also CMODS6.31, U$2.12; no longer CMODS6.10, ESP32.12
- net IO32: now also CMODS6.15, U$2.21; no longer CMODS6.41, ESP32.21
- net IO33: now also CMODS6.36, U$2.22; no longer CMODS6.42, ESP32.22
- net IO34: now also CMODS6.18, U$2.19; no longer CMODS6.39, ESP32.19
- net IO35: now also CMODS6.17, U$2.20; no longer CMODS6.40, ESP32.20
- net IO36: now also CMODS6.21, U$2.17; no longer CMODS6.37, ESP32.17
- net IO39: now also CMODS6.19, U$2.18; no longer CMODS6.38, ESP32.18
- net IO4: now also CMODS6.42, U$2.5; no longer CMODS6.3, ESP32.5
- net IO5: now also CMODS6.11, U$2.8; no longer CMODS6.6, ESP32.8
- net N$1: now also CMODS6.13; no longer CMODS6.36
- net N$10: now also IC2.12; no longer IC2.4
- net N$11: now also IC2.6; no longer IC2.2
- net N$12: now also IC2.4; no longer IC2.10
- net N$13: now also IC2.2; no longer IC2.12
- net N$15: now also IC3.10; no longer IC3.6
- net N$16: now also IC3.6; no longer IC3.4
- net N$17: now also IC3.4; no longer IC3.2
- net N$18: now also IC3.2; no longer IC3.10
- net N$24: now also IC4.12; no longer IC4.10
- net N$25: now also IC4.10; no longer IC4.12
- net N$3: now also IC1.2; no longer IC1.6
- net N$5: now also IC1.6; no longer IC1.2
- net N$6: now also IC1.12; no longer IC1.10
- net N$7: now also IC1.10; no longer IC1.12
- net N$9: now also IC2.10; no longer IC2.6
Routing:
- net N$8: track 0.00 -> 111.9 mm, vias 0 -> 1
- net N$9: track 0.00 -> 101.4 mm, vias 0 -> 1
- net N$11: track 0.00 -> 90.7 mm, vias 0 -> 1
- net IO3: track 0.00 -> 89.8 mm
- net N$10: track 0.00 -> 88.3 mm, vias 0 -> 1
- net IO16: track 0.00 -> 88.1 mm
- net IO21: track 0.00 -> 87.9 mm
- net IO4: track 0.00 -> 86.8 mm
- net IO19: track 0.00 -> 86.7 mm
- net IO2: track 0.00 -> 84.5 mm
- net IO17: track 0.00 -> 81.8 mm
- net IO23: track 0.00 -> 72.7 mm
- net IO18: track 0.00 -> 71.5 mm
- net IO22: track 0.00 -> 70.1 mm
- net N$1: track 0.00 -> 65.4 mm
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